Commit message: Add control do quimera_robot

File: urdf/quimera_robot.gazebo.xacro (robot description, xacro)
@@ -4,5 +4,5 @@
   <gazebo>
     <plugin name="gazebo_ros_control" filename="libgazebo_ros_control.so">
-      <robotNamespace>/mobile_robot</robotNamespace>
+      <robotNamespace>/quimera_robot</robotNamespace>
       <!--robotParam>/robot_description</robotParam-->
       <robotSimType>gazebo_ros_control/DefaultRobotHWSim</robotSimType>
@@ -30,3 +30,19 @@
     <xacro:set_wheel_friction link="front_right_wheel" friction="200"/>
   </xacro:macro>
+  <gazebo reference="back_left_wheel">
+    <material>Gazebo/Black</material>
+    <selfCollide>false</selfCollide>
+  </gazebo>
+  <gazebo reference="front_left_wheel">
+    <material>Gazebo/Red</material>
+    <selfCollide>false</selfCollide>
+  </gazebo>
+  <gazebo reference="back_right_wheel">
+    <material>Gazebo/Black</material>
+    <selfCollide>false</selfCollide>
+  </gazebo>
+  <gazebo reference="front_right_wheel">
+    <material>Gazebo/Red</material>
+    <selfCollide>false</selfCollide>
+  </gazebo>
 </robot>

Commit message: ros2 adjustments

File: urdf/quimera_robot.gazebo.xacro (robot description, xacro)
@@ -2,11 +2,49 @@
 <robot xmlns:xacro="http://ros.org/wiki/xacro">
   <!-- ros_control plugin -->
-  <gazebo>
+  <!-- <gazebo>
     <plugin name="gazebo_ros_control" filename="libgazebo_ros_control.so">
       <robotNamespace>/quimera_robot</robotNamespace>
-      <!--robotParam>/robot_description</robotParam-->
+      <robotParam>/robot_description</robotParam>
       <robotSimType>gazebo_ros_control/DefaultRobotHWSim</robotSimType>
-      <legacyModeNS>True</legacyModeNS>
     </plugin>
+  </gazebo> -->
+  <gazebo>
+    <plugin name="joint_states" filename="libgazebo_ros_joint_state_publisher.so">
+      <ros>
+        <!-- <namespace>/</namespace> -->
+          <argument>--ros-args</argument>
+          <argument>-r </argument>
+          <argument>~/out:=joint_states</argument>
+      </ros>
+      <update_rate>50</update_rate>
+      <joint_name>back_right_wheel_joint</joint_name>
+      <joint_name>back_left_wheel_joint</joint_name>
+      <joint_name>front_right_wheel_joint</joint_name>
+      <joint_name>front_left_wheel_joint</joint_name>
+    </plugin>
+    <plugin name="hoverboard_diff_drive" filename="libgazebo_ros_diff_drive.so">
+        <ros>
+          <!-- <namespace>/sim</namespace> -->
+          <remapping>cmd_vel:=/cmd_vel</remapping>
+        </ros>
+      <update_rate>50</update_rate>
+      <left_joint>back_left_wheel_joint</left_joint>
+      <right_joint>back_right_wheel_joint</right_joint>
+      <wheel_separation>0.073</wheel_separation>
+      <wheel_diameter>0.053</wheel_diameter>
+      <command_topic>cmd_vel</command_topic>
+      <!-- output -->
+      <publish_odom>true</publish_odom>
+      <publish_odom_tf>true</publish_odom_tf>
+      <publish_wheel_tf>true</publish_wheel_tf>
+      <odometry_topic>odom</odometry_topic>
+      <odometry_frame>odom</odometry_frame>
+      <robot_base_frame>base_footprint</robot_base_frame>
+      <max_wheel_torque>30</max_wheel_torque>
+      <max_wheel_acceleration>1.0</max_wheel_acceleration>
+    </plugin>
+  </gazebo>
+  <gazebo reference="base_link">
+    <material>Gazebo/White</material>
   </gazebo>
   <!-- xacro to set the friction for the wheel. This patch was taken from the MIR
@@ -30,19 +68,3 @@
     <xacro:set_wheel_friction link="front_right_wheel" friction="200"/>
   </xacro:macro>
-  <gazebo reference="back_left_wheel">
-    <material>Gazebo/Black</material>
-    <selfCollide>false</selfCollide>
-  </gazebo>
-  <gazebo reference="front_left_wheel">
-    <material>Gazebo/Red</material>
-    <selfCollide>false</selfCollide>
-  </gazebo>
-  <gazebo reference="back_right_wheel">
-    <material>Gazebo/Black</material>
-    <selfCollide>false</selfCollide>
-  </gazebo>
-  <gazebo reference="front_right_wheel">
-    <material>Gazebo/Red</material>
-    <selfCollide>false</selfCollide>
-  </gazebo>
 </robot>

File: urdf/quimera_robot.urdf.xacro (robot description, xacro)
@@ -1,9 +1,8 @@
 <?xml version="1.0"?>
 <robot xmlns:xacro="http://www.ros.org/wiki/xacro" name="quimera_robot">
-  <xacro:property name="package_name" value="mobile_robot_models"/>
-  <xacro:property name="package_lib" value="mobile_robot_description"/>
+  <xacro:property name="package_name" value="mobile_robot_description"/>
   <xacro:property name="robot_name" value="quimera_robot"/>
-  <xacro:include filename="$(find ${package_lib})/urdf/include/common_macros.urdf.xacro" />
-  <xacro:include filename="$(find ${package_lib})/urdf/include/common_sensors.xacro" />
+  <xacro:include filename="$(find ${package_name})/urdf/include/common_macros.urdf.xacro" />
+  <xacro:include filename="$(find ${package_name})/urdf/include/common_sensors.xacro" />
   <xacro:include filename="$(find ${package_name})/urdf/quimera_robot.gazebo.xacro" />
   <!-- <xacro:include filename="$(find hector_sensors_description)/urdf/generic_camera.urdf.xacro" /> -->
@@ -41,11 +40,12 @@
   </xacro:wheel>
   <!-- Sensors -->
-  <xacro:hokuyo_sensor parent_link="base_link" >
+  <xacro:hokuyo_sensor parent_link="base_link" visualize="false">
     <origin xyz="-0.02 0 ${base_props['base']['z_size'] + 0.05}" rpy="0 0 0" />
   </xacro:hokuyo_sensor>
-  <!-- <xacro:generic_camera name="camera" parent="base_link" ros_topic="image_raw"
-                        cam_info_topic="camera_info" update_rate="30"
-                        res_x="800" res_y="800" image_format="R8G8B8" h_fov="1.4" >
-        <origin xyz="0 0 0" rpy="0 0 0" />
-  </xacro:generic_camera>                       -->
+  <xacro:camera_sensor parent_link="base_link" visualize="false">
+    <origin xyz="0.02 0 ${base_props['base']['z_size']}" rpy="0 0 0" />
+  </xacro:camera_sensor>
+  <xacro:imu_sensor parent_link="base_link">
+    <origin xyz="0.0 0.05 ${base_props['base']['z_size'] + 0.01}" rpy="0 0 0" />
+  </xacro:imu_sensor>
 </robot>
